File: HW/EnvSensor/PAx5EnvSensor.sch (KiCad schematic (older format))
At the start: 42 parts, among them P1 PwrIn, P10 Photo, P11 USART, P12 ExtConn, P2 SWD, P20 Antenna, Q1 IRLML6402, SW1 SW-Push4, U1 STM32L051x-P, U20 RFM69HW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

Commit message: Coding and commenting style update
Parts:
- R52: value 4k -> 2k7
- R53: value 10k -> 330
Changed lines of the file:
@@
 P 2900 4900
 F 0 "R52" V 2980 4900 40  0000 C CNN
-F 1 "4k" V 2900 4900 40  0000 C CNN
+F 1 "2k7" V 2900 4900 40  0000 C CNN
 F 2 "Calin:R_1206_HandSoldering" V 2830 4900 30  0001 C CNN
 F 3 "" H 2900 4900 30  0000 C CNN
@@
 P 6550 4350
 F 0 "R53" V 6630 4350 40  0000 C CNN
-F 1 "10k" V 6550 4350 40  0000 C CNN
+F 1 "330" V 6550 4350 40  0000 C CNN
 F 2 "Calin:R_0805_HandSoldering" V 6480 4350 30  0001 C CNN
 F 3 "" H 6550 4350 30  0000 C CNN

Commit message: Archiving the repository
Parts:
- B1: footprint Calin:Box-Sens-LH-NPTH -> EnvSensor:Box-Sens-LH-NPTH; symbol BOARDLAYOUT -> EnvSensor:BOARDLAYOUT
- C1, C2, C20, C21, C3, C30, C4, C40, C41, C5, C50, C51, C6: footprint Calin:C_0805_HandSoldering -> EnvSensor:C_0805_HandSoldering; symbol C-PAx5 -> EnvSensor:C-PAx5
- D90: footprint Calin:LED_1206_HandSoldering -> EnvSensor:LED_1206_HandSoldering; symbol LED-PAx5 -> EnvSensor:LED-PAx5
- L1: footprint Calin:R_1206_HandSoldering -> EnvSensor:R_1206_HandSoldering; symbol INDUCTOR -> EnvSensor:INDUCTOR
- L40: footprint Calin:TYS50xx -> EnvSensor:TYS50xx; symbol INDUCTOR -> EnvSensor:INDUCTOR
- P1: footprint Calin:Pin_Header_Straight_1x02 -> EnvSensor:Pin_Header_Straight_1x02; symbol CS_2 -> EnvSensor:CS_2
- P10, P12, P2: footprint Calin:Pin_Header_Straight_1x04 -> EnvSensor:Pin_Header_Straight_1x04; symbol CS_4 -> EnvSensor:CS_4
- P11: footprint Calin:Pin_Header_Straight_1x03 -> EnvSensor:Pin_Header_Straight_1x03; symbol CS_3 -> EnvSensor:CS_3
- P20: footprint Calin:Pin_Header_Straight_1x01 -> EnvSensor:Pin_Header_Straight_1x01; symbol CS_1 -> EnvSensor:CS_1
- Po1, Po2: footprint Calin:PinTest-SMD -> EnvSensor:PinTest-SMD; symbol CS_1 -> EnvSensor:CS_1
- Q1: footprint Calin:SOT-23-calin -> EnvSensor:SOT-23-calin; symbol IRLML6402 -> EnvSensor:IRLML6402
- R1, R2, R3, R40, R41, R50, R51, R53: footprint Calin:R_0805_HandSoldering -> EnvSensor:R_0805_HandSoldering; symbol RR -> EnvSensor:RR
- R52, R90: footprint Calin:R_1206_HandSoldering -> EnvSensor:R_1206_HandSoldering; symbol RR -> EnvSensor:RR
- SW1: footprint Calin:cSW-Push-4 -> EnvSensor:cSW-Push-4; symbol SW-Push4 -> EnvSensor:SW-Push4
- U1: footprint Calin:cLQFP32-7-v2 -> EnvSensor:cLQFP32-7-v2; symbol STM32L051x-P -> EnvSensor:STM32L051x-P
- U20: footprint Calin:RFM69HW -> EnvSensor:RFM69HW; symbol RFM69HW -> EnvSensor:RFM69HW
- U30: footprint Calin:SOIC-8-N -> EnvSensor:SOIC-8-N; symbol M25P10-A -> EnvSensor:M25P10-A
- U40: footprint Calin:SOT23-6 -> EnvSensor:SOT23-6; symbol MCP16251 -> EnvSensor:MCP16251
- U50: footprint Calin:HIH8000 -> EnvSensor:HIH8000; symbol HIH8000_I2C -> EnvSensor:HIH8000_I2C
Connections:
- wire segments 179 -> 197
